Commit message: modification of the parts of the Link6 (connected to tibial plateau)

File: urdf/brace_bottom_setup.urdf (robot description, URDF)
Before this commit: robot brace_bottom_setup, 7 links, 6 joints
Links:
- link Link1: mass 1.50456576331701 -> 1.60283665795463
- link Link4: mass 0.374573654259201 -> 0.37932636432982
- link Link6: mass 0.099135009429078 -> 0.348002554128136
Joints:
- joint Joint5: origin xyz=0 0 0.545 rpy=0 0 0 -> xyz=0 0 0.495 rpy=0 0 0
- joint Joint6: origin xyz=0 0 0.0377480000000002 rpy=0 0 0 -> xyz=0 0 0.0377480000000001 rpy=0 0 0

Commit message: modification urdf bottom setup because issue in previous one with bottom force sensor

File: urdf/brace_bottom_setup.urdf (robot description, URDF)
Before this commit: robot brace_bottom_setup, 7 links, 6 joints
Joints:
- joint Joint4: origin xyz=-0.00199953015368963 0 0.01 rpy=0 0 0 -> xyz=-0.00199961697777845 0 0.01 rpy=0 0 0

Commit message: modification orientation force sensors bottom setup

File: urdf/brace_bottom_setup.urdf (robot description, URDF)
Before this commit: robot brace_bottom_setup, 7 links, 6 joints
Links:
- link Link5: mass 0.0185284683375794 -> 0.018528458539416
Joints:
- joint Joint3: origin xyz=0.00199999999999999 0 0.02425 rpy=0 0 0 -> xyz=-0.002 0 0.02425 rpy=0 0 0
- joint Joint4: origin xyz=-0.00199961697777845 0 0.01 rpy=0 0 0 -> xyz=0.00200008682408884 0 0.01 rpy=0 0 0
- joint Joint6: origin xyz=0 0 0.0377480000000001 rpy=0 0 0 -> xyz=0 0 0.0377479999999998 rpy=0 0 0

Commit message: modification of the thickness of the board and the length of the tibia tube

File: urdf/brace_bottom_setup.urdf (robot description, URDF)
Before this commit: robot brace_bottom_setup, 7 links, 6 joints
Links:
- link Link1: mass 1.60283665795463 -> 1.62139168956489
- link Link6: mass 0.348002554128136 -> 0.409264576522902
- link base_link: mass 0.748574502333434 -> 1.8963887392447
Joints:
- joint Joint4: origin xyz=0.00200008682408884 0 0.01 rpy=0 0 0 -> xyz=0.00200008682408884 0 0.0100000000000001 rpy=0 0 0
- joint Joint5: origin xyz=0 0 0.495 rpy=0 0 0 -> xyz=0 0 0.545 rpy=0 0 0
- joint Joint6: origin xyz=0 0 0.0377479999999998 rpy=0 0 0 -> xyz=0 0 0.037748 rpy=0 0 0

Commit message: modification origin base link

File: urdf/brace_bottom_setup.urdf (robot description, URDF)
Before this commit: robot brace_bottom_setup, 7 links, 6 joints
Joints:
- joint Joint1: origin xyz=0 0 0 rpy=0 0 0 -> xyz=0 0 0.038 rpy=0 0 0
- joint Joint2: origin xyz=0 0 0 rpy=0 0 0 -> xyz=0 0 0.038 rpy=0 0 0
- joint Joint6: origin xyz=0 0 0.037748 rpy=0 0 0 -> xyz=0 0 0.0377479999999999 rpy=0 0 0

Commit message: changing the anatomic axis for the brace_bottom_setup following the litterature

File: urdf/brace_bottom_setup.urdf (robot description, URDF)
Before this commit: robot brace_bottom_setup, 7 links, 6 joints
Links:
- link Link1: mass 1.62139168956489 -> 1.6213916895649
- link Link4: mass 0.37932636432982 -> 0.378986768395715
- link Link6: mass 0.409264576522902 -> 0.471343550095234
Joints:
- joint Joint6: origin xyz=0 0 0.0377479999999999 rpy=0 0 0 -> xyz=0.000479959249496128 0.0108570079505446 0.0577800157706738 rpy=0.0233655354660118 0.155971020087063 0.149323563771932

Commit message: restoring old urdf axis

File: urdf/brace_bottom_setup.urdf (robot description, URDF)
Before this commit: robot brace_bottom_setup, 7 links, 6 joints
Links:
- link Link1: mass 1.6213916895649 -> 1.62139168956489
- link Link4: mass 0.378986768395715 -> 0.37932636432982
- link Link6: mass 0.471343550095234 -> 0.409264576522902
Joints:
- joint Joint6: origin xyz=0.000479959249496128 0.0108570079505446 0.0577800157706738 rpy=0.0233655354660118 0.155971020087063 0.149323563771932 -> xyz=0 0 0.0377479999999999 rpy=0 0 0

Commit message: modif plaque tibia

File: urdf/brace_bottom_setup.urdf (robot description, URDF)
Before this commit: robot brace_bottom_setup, 7 links, 6 joints
Links:
- link Link4: mass 0.37932636432982 -> 0.378986768395715
- link Link6: mass 0.409264576522902 -> 0.334059103128422
Joints:
- joint Joint3: origin xyz=-0.002 0 0.02425 rpy=0 0 0 -> xyz=-0.00200000000000001 0 0.02425 rpy=0 0 0
- joint Joint4: origin xyz=0.00200008682408884 0 0.0100000000000001 rpy=0 0 0 -> xyz=0.00200008682408882 0 0.01 rpy=0 0 0
- joint Joint6: origin xyz=0 0 0.0377479999999999 rpy=0 0 0 -> xyz=0 0 0.037748 rpy=0 0 0

Commit message: corrections because errors

File: urdf/brace_bottom_setup.urdf (robot description, URDF)
Before this commit: robot brace_bottom_setup, 7 links, 6 joints
Links:
- link Link1: mass 1.62139168956489 -> 0.466390967517534
- link Link2: mass 0.0776928177876513 -> 0.0787348629786105
- link Link3: mass 0.018528458539416 -> 0.0185862462856871
- link Link4: mass 0.378986768395715 -> 0.612322959263128
- link Link5: mass 0.018528458539416 -> 0.0185862466941427
- link Link6: mass 0.334059103128422 -> 0.270541546668934
- link base_link: mass 1.8963887392447 -> 2.24707410283585
Joints:
- joint Joint1: origin xyz=0 0 0.038 rpy=0 0 0 -> xyz=0.00346392795414539 0.117367542402842 0.841449957714373 rpy=1.5707963267949 -1.41769797329821 0
- joint Joint2: origin xyz=0 0 0.038 rpy=0 0 0 -> xyz=-0.1975517853149 -0.162632485347158 0.850207481202172 rpy=1.5707963267949 -1.41769797329821 0
- joint Joint3: origin xyz=-0.00200000000000001 0 0.02425 rpy=0 0 0 -> xyz=-0.0220204740295852 0.214998906537437 0.0149999999999998 rpy=0 0 0; parent Link2 -> Link1
- joint Joint4: origin xyz=0.00200008682408882 0 0.01 rpy=0 0 0 -> xyz=2.00211044838472E-05 0 0.015748 rpy=0 0 0
- joint Joint5: origin xyz=0 0 0.545 rpy=0 0 0 -> xyz=0 0 0.015 rpy=0 0 0; parent Link1 -> Link2
- joint Joint6: origin xyz=0 0 0.037748 rpy=0 0 0 -> xyz=-0.0050213656357877 0.0050209600560045 0.015748 rpy=0 0 0

Commit message: changing the base link coordinate system

File: urdf/brace_bottom_setup.urdf (robot description, URDF)
Before this commit: robot brace_bottom_setup, 7 links, 6 joints
Links:
- link Link1: mass 0.466390967517534 -> 0.466390967517537
- link Link4: mass 0.612322959263128 -> 1.25386550462557
Joints:
- joint Joint1: origin xyz=0.00346392795414539 0.117367542402842 0.841449957714373 rpy=1.5707963267949 -1.41769797329821 0 -> xyz=-0.00299998465083984 0.0161999548741417 0.215000000000001 rpy=0 0 0
- joint Joint2: origin xyz=-0.1975517853149 -0.162632485347158 0.850207481202172 rpy=1.5707963267949 -1.41769797329821 0 -> xyz=-0.024999986892059 0.216199935816294 0.49500002775 rpy=0 0 0
- joint Joint3: origin xyz=-0.0220204740295852 0.214998906537437 0.0149999999999998 rpy=0 0 0 -> xyz=-0.0220204740295803 0.21499890653722 0.0149999999999984 rpy=0 0 0
- joint Joint6: origin xyz=-0.0050213656357877 0.0050209600560045 0.015748 rpy=0 0 0 -> xyz=-0.00502055183810024 0.00502049020968376 0.0157480000000001 rpy=0 0 0

Commit message: changing the part under the tibial plateau (holes for the cones calib part) + modification of the position of the brace on the calf

File: urdf/brace_bottom_setup.urdf (robot description, URDF)
Before this commit: robot brace_bottom_setup, 7 links, 6 joints
Links:
- link Link1: mass 0.466390967517537 -> 0.466390967517536
- link Link4: mass 1.25386550462557 -> 1.25386550398595
Joints:
- joint Joint1: origin xyz=-0.00299998465083984 0.0161999548741417 0.215000000000001 rpy=0 0 0 -> xyz=0.0034639279539304 0.117367542402841 0.841449957714401 rpy=1.5707963267949 -1.41769797329821 0
- joint Joint2: origin xyz=-0.024999986892059 0.216199935816294 0.49500002775 rpy=0 0 0 -> xyz=-0.197551740096197 -0.162632464134194 0.850207474224662 rpy=1.5707963267949 -1.41769797329821 0
- joint Joint6: origin xyz=-0.00502055183810024 0.00502049020968376 0.0157480000000001 rpy=0 0 0 -> xyz=-0.00502055183811378 0.0050204902097179 0.0157479999999958 rpy=0 0 0

Commit message: modif pour ajouter les plaques des sensors des forces shoes

File: urdf/brace_bottom_setup.urdf (robot description, URDF)
Before this commit: robot brace_bottom_setup, 7 links, 6 joints
Links:
- link Link1: mass 0.466390967517536 -> 0.493518956002241
- link Link2: mass 0.0787348629786105 -> 0.105862851463318
- link Link4: mass 1.25386550398595 -> 0.633705360714929
- link Link5: mass 0.0185862466941427 -> 0.0185862466941426
- link Link6: mass 0.270541546668934 -> 0.291923645802481
Joints:
- joint Joint1: origin xyz=0.0034639279539304 0.117367542402841 0.841449957714401 rpy=1.5707963267949 -1.41769797329821 0 -> xyz=0.0195000022412237 0.00960000406644995 0.161251997758775 rpy=0 0 0
- joint Joint2: origin xyz=-0.197551740096197 -0.162632464134194 0.850207474224662 rpy=1.5707963267949 -1.41769797329821 0 -> xyz=-0.00249999999999495 0.209599976316459 0.495000027749999 rpy=0 0 0
- joint Joint3: origin xyz=-0.0220204740295803 0.21499890653722 0.0149999999999984 rpy=0 0 0 -> xyz=-0.0170196602318987 0.19999928955966 0.02 rpy=0 0 0
- joint Joint4: origin xyz=2.00211044838472E-05 0 0.015748 rpy=0 0 0 -> xyz=-0.0158146026210939 0 0.0197480000000001 rpy=0 0 0
- joint Joint6: origin xyz=-0.00502055183811378 0.0050204902097179 0.0157479999999958 rpy=0 0 0 -> xyz=-0.00712040356960131 -0.00135982032125276 0.0247480000000005 rpy=0 0 0

Commit message: changing base_link_CS definition

File: urdf/brace_bottom_setup.urdf (robot description, URDF)
Before this commit: robot brace_bottom_setup, 7 links, 6 joints
Links:
- link Link4: mass 0.633705360714929 -> 0.633705058396686
Joints:
- joint Joint1: origin xyz=0.0195000022412237 0.00960000406644995 0.161251997758775 rpy=0 0 0 -> xyz=-0.00960000406645026 -0.161251997758775 0.0195000022412237 rpy=1.5707963267949 -1.5707963267949 0
- joint Joint2: origin xyz=-0.00249999999999495 0.209599976316459 0.495000027749999 rpy=0 0 0 -> xyz=-0.209599976316459 -0.49500002775 -0.00249999999999917 rpy=1.5707963267949 -1.5707963267949 0
- joint Joint6: origin xyz=-0.00712040356960131 -0.00135982032125276 0.0247480000000005 rpy=0 0 0 -> xyz=-0.00712040356960109 -0.00135982032125259 0.0247480000000004 rpy=0 0 0
